Commit message: 🎈 perf: 修改为相对路径；使用xacro

File: src/ranger_mini_v2_gazebo/xacro/ranger_mini_gazebo.xacro (robot description, xacro)
@@ -29,5 +29,5 @@
             <origin xyz="0 0 0" rpy="1.57 0 3.14 " />
             <geometry>
-                <mesh filename="package://ranger_mini_v2/meshes/ranger_base.dae" />
+                <mesh filename="file://$(find ranger_mini_v2)/meshes/ranger_base.dae" />
             </geometry>
         </visual>
@@ -48,5 +48,5 @@
             <origin xyz="-0.23 -0.194 0.1" rpy="1.57 0 3.14 " />
             <geometry>
-                    <mesh filename="package://ranger_mini_v2/meshes/fl.dae" />
+                <mesh filename="file://$(find ranger_mini_v2)/meshes/fl.dae" />
             </geometry>
         </visual>
@@ -110,5 +110,5 @@
             <origin xyz="-0.23 0.194 0.1" rpy="1.57 0 3.14 " />
             <geometry>
-                <mesh filename="package://ranger_mini_v2/meshes/fr.dae" />
+                <mesh filename="file://$(find ranger_mini_v2)/meshes/fr.dae" />
             </geometry>
         </visual>
@@ -166,5 +166,5 @@
             <origin xyz="-0.23 -0.194 0.1" rpy="1.57 0 3.14 " />
             <geometry>
-                    <mesh filename="package://ranger_mini_v2/meshes/fl.dae" />
+                <mesh filename="file://$(find ranger_mini_v2)/meshes/fl.dae" />
             </geometry>
         </visual>
@@ -222,5 +222,5 @@
             <origin xyz="-0.23 0.194 0.1" rpy="1.57 0 3.14 " />
             <geometry>
-                    <mesh filename="package://ranger_mini_v2/meshes/fr.dae" />
+                    <mesh filename="file://$(find ranger_mini_v2)/meshes/fr.dae" />
             </geometry>
         </visual>
@@ -269,18 +269,20 @@
             <axis xyz="0 1 0" rpy="0 0 0" />
         </joint>
-    <plugin name="ranger_mini_joint_state" filename="libgazebo_ros_joint_state_publisher.so">
-      <ros>
-          <remapping>~/out:=joint_states</remapping>
-      </ros>
-      <update_rate>30</update_rate>
-      <joint_name>fl_wheel</joint_name>
-      <joint_name>fr_wheel</joint_name>
-      <joint_name>rl_wheel</joint_name>
-      <joint_name>rr_wheel</joint_name>
-      <joint_name>fl_steering_wheel</joint_name>
-      <joint_name>fr_steering_wheel</joint_name>
-      <joint_name>rl_steering_wheel</joint_name>
-      <joint_name>rr_steering_wheel</joint_name>
-    </plugin>
+    <gazebo>
+        <plugin name="ranger_mini_joint_state" filename="libgazebo_ros_joint_state_publisher.so">
+        <ros>
+            <remapping>~/out:=joint_states</remapping>
+        </ros>
+        <update_rate>30</update_rate>
+        <joint_name>fl_wheel</joint_name>
+        <joint_name>fr_wheel</joint_name>
+        <joint_name>rl_wheel</joint_name>
+        <joint_name>rr_wheel</joint_name>
+        <joint_name>fl_steering_wheel</joint_name>
+        <joint_name>fr_steering_wheel</joint_name>
+        <joint_name>rl_steering_wheel</joint_name>
+        <joint_name>rr_steering_wheel</joint_name>
+        </plugin>
+    </gazebo>
     <ros2_control name="GazeboSystem" type="system">
         <hardware>
@@ -364,6 +366,8 @@
         </joint>
     </ros2_control>
-    <plugin name="gazebo_ros2_control" filename="libgazebo_ros2_control.so">
-        <parameters>/home/nvidia/ranger_mini_v2/install/ranger_mini_v2/share/ranger_mini_v2/config/controllers.yaml</parameters>
-    </plugin>
+    <gazebo>
+        <plugin name="gazebo_ros2_control" filename="libgazebo_ros2_control.so">
+            <parameters>$(find ranger_mini_v2)/config/controllers.yaml</parameters>
+        </plugin>
+    </gazebo>
 </robot>

File: src/ranger_mini_v2_gazebo/xacro/ranger_mini_real.xacro (robot description, xacro)
@@ -29,5 +29,5 @@
             <origin xyz="0 0 0" rpy="1.57 0 3.14 " />
             <geometry>
-                <mesh filename="package://ranger_mini_v2/meshes/ranger_base.dae" />
+                <mesh filename="file://$(find ranger_mini_v2)/meshes/ranger_base.dae" />
             </geometry>
         </visual>
@@ -48,5 +48,5 @@
             <origin xyz="-0.23 -0.194 0.1" rpy="1.57 0 3.14 " />
             <geometry>
-                    <mesh filename="package://ranger_mini_v2/meshes/fl.dae" />
+                    <mesh filename="file://$(find ranger_mini_v2)/meshes/fl.dae" />
             </geometry>
         </visual>
@@ -110,5 +110,5 @@
             <origin xyz="-0.23 0.194 0.1" rpy="1.57 0 3.14 " />
             <geometry>
-                <mesh filename="package://ranger_mini_v2/meshes/fr.dae" />
+                <mesh filename="file://$(find ranger_mini_v2)/meshes/fr.dae" />
             </geometry>
         </visual>
@@ -166,5 +166,5 @@
             <origin xyz="-0.23 -0.194 0.1" rpy="1.57 0 3.14 " />
             <geometry>
-                    <mesh filename="package://ranger_mini_v2/meshes/fl.dae" />
+                    <mesh filename="file://$(find ranger_mini_v2)/meshes/fl.dae" />
             </geometry>
         </visual>
@@ -222,5 +222,5 @@
             <origin xyz="-0.23 0.194 0.1" rpy="1.57 0 3.14 " />
             <geometry>
-                    <mesh filename="package://ranger_mini_v2/meshes/fr.dae" />
+                    <mesh filename="file://$(find ranger_mini_v2)/meshes/fr.dae" />
             </geometry>
         </visual>
